Commit message: added the create ws

File: test_rviz3/src/jetson_bot_urdf/urdf/jetson_bot_urdf.urdf (robot description, URDF)
Before this commit: robot jetson_bot_urdf, 7 links, 6 joints
Links:
- removed link camera_depth_frame
- removed link camera_depth_optical_frame
- removed link camera_rgb_frame
- removed link camera_rgb_optical_frame
Joints:
- removed joint cdf_joint
- removed joint cdof_joint
- removed joint crf_joint
- removed joint crof_joint
